Commit message: reorganized launch files, tweaked urdf

File: urdf/ninjacar.urdf.xacro (robot description, xacro)
@@ -1,22 +1,32 @@
 <?xml version="1.0"?>
 <robot name="ninjacar" xmlns:xacro="http://ros.org/wiki/xacro">
+  <link name="imu_link"/>
+  <link name="body_aligned_imu_link"/>
+  <joint name="aligned_imu" type="fixed">
+  <parent link="body_aligned_imu_link" />
+    <child link="imu_link" />
+    <origin xyz="0 0 0" rpy="0 0 -1.570796325" />
+  </joint>
   <link name="xavier"/> <!-- centroid of heat sink projected to footprint -->
-  <joint name="xavier_ouster" type="fixed">
+  <!-- <joint name="xavier_ouster" type="fixed">
     <parent link="xavier" />
     <child link="os1_sensor" />
     <origin xyz="0.1157614 0 0.0329911" rpy="0 0 -1.570796325" />
   </joint>
-  <link name="os1_sensor"/>
-  <link name="imu_link"/>
-  <link name="body_aligned_imu_link"/>
+  <link name="os1_sensor"/> -->
+  <!-- <xacro:include filename="$(find ouster_ros)/OS1-64.urdf.xacro"/>
+  <OS1-64 parent="xavier">
+    <origin xyz="0.1157614 0 0.0329911" rpy="0 0 -1.570796325" />
+  </OS1-64> -->
+  <!-- <joint name="ouster" type="fixed">
+    <parent link="os1_sensor" />
+    <child link="os1_lidar" />
+    <origin xyz="0 0 0.03816" rpy="0 0 -3.14159265" />
+  </joint> -->
+  <!-- <link name="os1_sensor"/> -->
   <joint name="xavier_imu" type="fixed">
-    <parent link="xavier" />
-    <child link="imu_link" />
-    <origin xyz="0.1154054 0 -0.0077934 " rpy="0 0 1.570796325" />
-  </joint>
-  <joint name="aligned_imu" type="fixed">
-    <parent link="imu_link" />
-    <child link="body_aligned_imu_link" />
-    <origin xyz="0 0 0" rpy="0 0 -1.570796325" />
+    <parent link="body_aligned_imu_link" />
+    <child link="xavier" />
+    <origin xyz="-0.1154054 0 0.0077934 " rpy="0 0 0" />
   </joint>
   <!-- <joint name="ouster_imu" type="fixed">
@@ -25,7 +35,49 @@
     <origin xyz="0.1971268 0 -0.0007798" rpy="0 0 0" />
   </joint> -->
-  <xacro:include filename="$(find realsense2_description)/urdf/_d435.urdf.xacro"/>
-  <sensor_d435 parent="xavier" name="camera" >
+  <xacro:include filename="$(find realsense2_camera)/urdf/_d435.urdf.xacro"/>
+  <link name="camera_fwd"/>
+  <joint name="camera_fwd" type="fixed">
+    <parent link="xavier" />
+    <child link="camera_fwd" />
+    <origin xyz="0.2219971 0 0.0130257" rpy="0 0 0" />
+  </joint>
+  <sensor_d435 parent="camera_fwd">
+    <origin xyz="0 0 0" rpy="0 0 0" />
+  </sensor_d435>
+  <link name="camera_low"/>
+  <joint name="camera_low" type="fixed">
+    <parent link="camera_fwd" />
+    <child link="camera_low" />
+    <origin xyz="-0.0136486 0 -0.0366877" rpy="0 0.523599 0" />
+  </joint>
+  <sensor_d435 parent="camera_low">
+    <origin xyz="0 0 0" rpy="0 0 0" />
+  </sensor_d435>
+<!-- OUSTER -->
+  <joint name="mount_joint" type="fixed">
+    <parent link="xavier"/>
+    <child link="os1_sensor"/>
     <origin xyz="0.1971268 0 -0.0007798" rpy="0 0 0" />
-  </sensor_d435>
+  </joint>
+  <link name="os1_sensor">
+    <visual name="base_visual">
+       <origin xyz="0 0 0.0" rpy="0 0 1.5707" />
+       <geometry>
+         <!-- <mesh filename="package://ouster_description/meshes/os1_64.dae" /> -->
+         <cylinder length="0.073" radius="0.04" />
+       </geometry>
+    </visual>
+  </link>
+  <link name="os1_imu" />
+  <link name="os1_lidar" />
+  <joint name="imu_link_joint" type="fixed">
+    <parent link="os1_sensor" />
+    <child link="os1_imu" />
+    <origin xyz="0.006253 -0.011775 0.007645" rpy="0 0 0" />
+  </joint>
+  <joint name="lidar_link_joint" type="fixed">
+    <parent link="os1_sensor" />
+    <child link="os1_lidar" />
+    <origin xyz="0.0 0.0 0.03618" rpy="0 0 3.14159265" />
+  </joint>
 </robot>

Commit message: added a bunch of stuff related to development of mochaplanner and mochavehicle

File: urdf/ninjacar.urdf.xacro (robot description, xacro)
@@ -1,4 +1,7 @@
 <?xml version="1.0"?>
 <robot name="ninjacar" xmlns:xacro="http://ros.org/wiki/xacro">
+  <material name="aluminum">
+	  <color rgba="0.5 0.5 0.5 1"/>
+    </material>
   <link name="imu_link"/>
   <link name="body_aligned_imu_link"/>
@@ -35,6 +38,6 @@
     <origin xyz="0.1971268 0 -0.0007798" rpy="0 0 0" />
   </joint> -->
-  <xacro:include filename="$(find realsense2_camera)/urdf/_d435.urdf.xacro"/>
-  <link name="camera_fwd"/>
+  <xacro:include filename="$(find realsense2_description)/urdf/_d435.urdf.xacro"/>
+  <!-- <link name="camera_fwd"/>
   <joint name="camera_fwd" type="fixed">
     <parent link="xavier" />
@@ -53,4 +56,10 @@
   <sensor_d435 parent="camera_low">
     <origin xyz="0 0 0" rpy="0 0 0" />
+  </sensor_d435> -->
+  <sensor_d435 parent="xavier" name="camera_fwd">
+    <origin xyz="0.2219971 0 0.0130257" rpy="0 0 0" />
+  </sensor_d435>
+  <sensor_d435 parent="camera_fwd_bottom_screw_frame" name="camera_low">
+    <origin xyz="-0.0136486 0 -0.0366877" rpy="0 0.523599 0" />
   </sensor_d435>
 <!-- OUSTER -->

Commit message: setup sensors/vicon/urdf for structured experiments, throttled/removed prints

File: urdf/ninjacar.urdf.xacro (robot description, xacro)
@@ -1,8 +1,8 @@
 <?xml version="1.0"?>
 <robot name="ninjacar" xmlns:xacro="http://ros.org/wiki/xacro">
-  <material name="aluminum">
+  <!-- <material name="aluminum">
 	  <color rgba="0.5 0.5 0.5 1"/>
-    </material>
-  <link name="imu_link"/>
+    </material> -->
+  <!-- <link name="imu_link"/>
   <link name="body_aligned_imu_link"/>
   <joint name="aligned_imu" type="fixed">
@@ -10,83 +10,14 @@
     <child link="imu_link" />
     <origin xyz="0 0 0" rpy="0 0 -1.570796325" />
-  </joint>
-  <link name="xavier"/> <!-- centroid of heat sink projected to footprint -->
-  <!-- <joint name="xavier_ouster" type="fixed">
-    <parent link="xavier" />
-    <child link="os1_sensor" />
-    <origin xyz="0.1157614 0 0.0329911" rpy="0 0 -1.570796325" />
-  </joint>
-  <link name="os1_sensor"/> -->
-  <!-- <xacro:include filename="$(find ouster_ros)/OS1-64.urdf.xacro"/>
-  <OS1-64 parent="xavier">
-    <origin xyz="0.1157614 0 0.0329911" rpy="0 0 -1.570796325" />
-  </OS1-64> -->
-  <!-- <joint name="ouster" type="fixed">
-    <parent link="os1_sensor" />
-    <child link="os1_lidar" />
-    <origin xyz="0 0 0.03816" rpy="0 0 -3.14159265" />
   </joint> -->
-  <!-- <link name="os1_sensor"/> -->
-  <joint name="xavier_imu" type="fixed">
+  <link name="N01/base_link"/>
+  <!-- <joint name="cpu_imu" type="fixed">
     <parent link="body_aligned_imu_link" />
-    <child link="xavier" />
+    <child link="cpu" />
     <origin xyz="-0.1154054 0 0.0077934 " rpy="0 0 0" />
-  </joint>
-  <!-- <joint name="ouster_imu" type="fixed">
-    <parent link="xavier" />
-    <child link="camera" />
-    <origin xyz="0.1971268 0 -0.0007798" rpy="0 0 0" />
   </joint> -->
   <xacro:include filename="$(find realsense2_description)/urdf/_d435.urdf.xacro"/>
-  <!-- <link name="camera_fwd"/>
-  <joint name="camera_fwd" type="fixed">
-    <parent link="xavier" />
-    <child link="camera_fwd" />
-    <origin xyz="0.2219971 0 0.0130257" rpy="0 0 0" />
-  </joint>
-  <sensor_d435 parent="camera_fwd">
-    <origin xyz="0 0 0" rpy="0 0 0" />
-  </sensor_d435>
-  <link name="camera_low"/>
-  <joint name="camera_low" type="fixed">
-    <parent link="camera_fwd" />
-    <child link="camera_low" />
-    <origin xyz="-0.0136486 0 -0.0366877" rpy="0 0.523599 0" />
-  </joint>
-  <sensor_d435 parent="camera_low">
-    <origin xyz="0 0 0" rpy="0 0 0" />
-  </sensor_d435> -->
-  <sensor_d435 parent="xavier" name="camera_fwd">
+  <sensor_d435 parent="N01/base_link" name="camera">
     <origin xyz="0.2219971 0 0.0130257" rpy="0 0 0" />
   </sensor_d435>
-  <sensor_d435 parent="camera_fwd_bottom_screw_frame" name="camera_low">
-    <origin xyz="-0.0136486 0 -0.0366877" rpy="0 0.523599 0" />
-  </sensor_d435>
-<!-- OUSTER -->
-  <joint name="mount_joint" type="fixed">
-    <parent link="xavier"/>
-    <child link="os1_sensor"/>
-    <origin xyz="0.1971268 0 -0.0007798" rpy="0 0 0" />
-  </joint>
-  <link name="os1_sensor">
-    <visual name="base_visual">
-       <origin xyz="0 0 0.0" rpy="0 0 1.5707" />
-       <geometry>
-         <!-- <mesh filename="package://ouster_description/meshes/os1_64.dae" /> -->
-         <cylinder length="0.073" radius="0.04" />
-       </geometry>
-    </visual>
-  </link>
-  <link name="os1_imu" />
-  <link name="os1_lidar" />
-  <joint name="imu_link_joint" type="fixed">
-    <parent link="os1_sensor" />
-    <child link="os1_imu" />
-    <origin xyz="0.006253 -0.011775 0.007645" rpy="0 0 0" />
-  </joint>
-  <joint name="lidar_link_joint" type="fixed">
-    <parent link="os1_sensor" />
-    <child link="os1_lidar" />
-    <origin xyz="0.0 0.0 0.03618" rpy="0 0 3.14159265" />
-  </joint>
 </robot>

Commit message: added launchfiles/urdfs for ninjacar experiments (mapping, sensors, mocap)

File: urdf/ninjacar.urdf.xacro (robot description, xacro)
@@ -11,5 +11,6 @@
     <origin xyz="0 0 0" rpy="0 0 -1.570796325" />
   </joint> -->
-  <link name="N01/base_link"/>
+  <link name="base_link"/>
+  <link name="royale_camera_link"/>
   <!-- <joint name="cpu_imu" type="fixed">
     <parent link="body_aligned_imu_link" />
@@ -18,6 +19,11 @@
   </joint> -->
   <xacro:include filename="$(find realsense2_description)/urdf/_d435.urdf.xacro"/>
-  <sensor_d435 parent="N01/base_link" name="camera">
+  <sensor_d435 parent="base_link" name="rs_camera">
     <origin xyz="0.2219971 0 0.0130257" rpy="0 0 0" />
   </sensor_d435>
+  <joint name="royale_cam_joint" type="fixed">
+    <parent link="base_link" />
+    <child link="royale_camera_link" />
+    <origin xyz="0.2219971 0 0.0130257" rpy="0 0 0" />
+  </joint>
 </robot>

Commit message: cleaned up, added microstrain/ouster launches, updated urdf

File: urdf/ninjacar.urdf.xacro (robot description, xacro)
@@ -11,19 +11,45 @@
     <origin xyz="0 0 0" rpy="0 0 -1.570796325" />
   </joint> -->
-  <link name="base_link"/>
-  <link name="royale_camera_link"/>
-  <!-- <joint name="cpu_imu" type="fixed">
-    <parent link="body_aligned_imu_link" />
-    <child link="cpu" />
-    <origin xyz="-0.1154054 0 0.0077934 " rpy="0 0 0" />
+  <link name="base_link"/> <!-- co-located/-oriented with bottom_plate_link -->
+  <link name="bottom_plate_link"/>  <!-- at xy center of vehicle, z at bottom of bottom plate -->
+  <joint name="bottom_plate_joint" type="fixed">
+    <parent link="base_link" />
+    <child link="bottom_plate_link" />
+    <origin xyz="0 0 0" rpy="0 0 0" />
+  </joint>
+  <link name="top_plate_link"/>  <!-- at xy center of vehicle, z at top of top plate -->
+  <joint name="top_plate_joint" type="fixed">
+    <parent link="bottom_plate_link" />
+    <child link="top_plate_link" />
+    <origin xyz="0 0 0.135" rpy="0 0 0" />
+  </joint>
+  <link name="os_sensor"/> <!-- lidar sensor frame -->
+  <joint name="os_joint" type="fixed">
+    <parent link="top_plate_link" />
+    <child link="os_sensor" />
+    <origin xyz="0.0387309 0 0" rpy="0 0 -1.5708" />
+  </joint>
+  <!-- body-aligned colocated with gx5_link -->
+  <!-- <link name="imu_link"/>
+  <joint name="imu_joint" type="fixed">
+    <parent link="top_plate_link" />
+    <child link="imu_link" />
+    <origin xyz="0.0387309 0 0" rpy="0 0 0" />
   </joint> -->
+  <link name="gx5_link"/> <!-- imu sensor frame -->
+  <joint name="gx5_joint" type="fixed">
+    <parent link="os_sensor" />
+    <child link="gx5_link" />
+    <origin xyz="0 0 -0.007675" rpy="0 0 3.1416" />
+  </joint>
   <xacro:include filename="$(find realsense2_description)/urdf/_d435.urdf.xacro"/>
-  <sensor_d435 parent="base_link" name="rs_camera">
+  <sensor_d435 parent="top_plate_link" name="rs_camera">
     <origin xyz="0.2219971 0 0.0130257" rpy="0 0 0" />
   </sensor_d435>
+  <link name="royale_camera_link"/>
   <joint name="royale_cam_joint" type="fixed">
-    <parent link="base_link" />
+    <parent link="top_plate_link" />
     <child link="royale_camera_link" />
-    <origin xyz="0.2219971 0 0.0130257" rpy="0 0 0" />
+    <origin xyz="0.2219971 0 0.0130257" rpy="3.1416 0 0" />
   </joint>
 </robot>

Commit message: added WayPoints msg, added liosam/vicon/static/fake localization and infinitam and sensors/ouster to launchfiles, moved vicon_demo launchfile to vicon_tools pkg, updated rviz file, updated urdf

File: urdf/ninjacar.urdf.xacro (robot description, xacro)
@@ -47,9 +47,15 @@
     <origin xyz="0.2219971 0 0.0130257" rpy="0 0 0" />
   </sensor_d435>
+  <link name="depth_camera_link"/>
+  <joint name="depth_cam_joint" type="fixed">
+    <parent link="top_plate_link" />
+    <child link="depth_camera_link" />
+    <origin xyz="0.2219971 0 0.0130257" rpy="0 0 0" />
+  </joint>
   <link name="royale_camera_link"/>
   <joint name="royale_cam_joint" type="fixed">
-    <parent link="top_plate_link" />
+    <parent link="depth_camera_link" />
     <child link="royale_camera_link" />
-    <origin xyz="0.2219971 0 0.0130257" rpy="3.1416 0 0" />
+    <origin xyz="0 0 0" rpy="3.1415 0 3.1415" />
   </joint>
 </robot>

Commit message: added joy_goal_generator, renamed a couple ambiguous tools, added depth completion options to launchfiles, updated urdf

File: urdf/ninjacar.urdf.xacro (robot description, xacro)
@@ -12,15 +12,21 @@
   </joint> -->
   <link name="base_link"/> <!-- co-located/-oriented with bottom_plate_link -->
-  <link name="bottom_plate_link"/>  <!-- at xy center of vehicle, z at bottom of bottom plate -->
-  <joint name="bottom_plate_joint" type="fixed">
+  <link name="top_plate_link"/> <!-- at xy center of vehicle, z at top of top plate -->
+  <joint name="top_plate_joint" type="fixed">
     <parent link="base_link" />
-    <child link="bottom_plate_link" />
+    <child link="top_plate_link" />
     <origin xyz="0 0 0" rpy="0 0 0" />
   </joint>
-  <link name="top_plate_link"/>  <!-- at xy center of vehicle, z at top of top plate -->
-  <joint name="top_plate_joint" type="fixed">
+  <link name="bottom_plate_link"/> <!-- at xy center of vehicle, z at bottom of bottom plate -->
+  <joint name="bottom_plate_joint" type="fixed">
+    <parent link="top_plate_link" />
+    <child link="bottom_plate_link" />
+    <origin xyz="0 0 -0.135" rpy="0 0 0" />
+  </joint>
+  <link name="footprint_link"/> <!-- at xy center of vehicle, z at bottom of wheels at neutral suspension -->
+  <joint name="footprint_joint" type="fixed">
     <parent link="bottom_plate_link" />
-    <child link="top_plate_link" />
-    <origin xyz="0 0 0.135" rpy="0 0 0" />
+    <child link="footprint_link" />
+    <origin xyz="0 0 -0.060" rpy="0 0 0" />
   </joint>
   <link name="os_sensor"/> <!-- lidar sensor frame -->

Commit message: switched to realsense depth, added waypoints params, added vicon tf comparison, added joy waypoint generator

File: urdf/ninjacar.urdf.xacro (robot description, xacro)
@@ -22,5 +22,5 @@
     <parent link="top_plate_link" />
     <child link="bottom_plate_link" />
-    <origin xyz="0 0 -0.135" rpy="0 0 0" />
+    <origin xyz="0 0 -0.127" rpy="0 0 0" />
   </joint>
   <link name="footprint_link"/> <!-- at xy center of vehicle, z at bottom of wheels at neutral suspension -->
@@ -49,13 +49,10 @@
     <origin xyz="0 0 -0.007675" rpy="0 0 3.1416" />
   </joint>
-  <xacro:include filename="$(find realsense2_description)/urdf/_d435.urdf.xacro"/>
-  <sensor_d435 parent="top_plate_link" name="rs_camera">
-    <origin xyz="0.2219971 0 0.0130257" rpy="0 0 0" />
-  </sensor_d435>
   <link name="depth_camera_link"/>
   <joint name="depth_cam_joint" type="fixed">
     <parent link="top_plate_link" />
     <child link="depth_camera_link" />
-    <origin xyz="0.2219971 0 0.0130257" rpy="0 0 0" />
+    <!-- <origin xyz="0.2219971 0 0.130257" rpy="0 0 0" /> -->
+    <origin xyz="0.1143 0 0.13335" rpy="0 0 0" />
   </joint>
   <link name="royale_camera_link"/>
@@ -63,5 +60,15 @@
     <parent link="depth_camera_link" />
     <child link="royale_camera_link" />
-    <origin xyz="0 0 0" rpy="3.1415 0 3.1415" />
+    <origin xyz="0 0 0" rpy="0 0 3.1415" />
+  </joint>
+  <xacro:include filename="$(find realsense2_description)/urdf/_d435.urdf.xacro"/>
+  <sensor_d435 parent="depth_camera_link" name="d435_camera">
+    <origin xyz="0 0 -0.0127" rpy="0 0 0" />
+  </sensor_d435>
+  <link name="t265_link"/>
+  <joint name="t265_camera_joint" type="fixed">
+    <parent link="top_plate_link" />
+    <child link="t265_link" />
+    <origin xyz="0.0254 0 0.1143" rpy="3.1415 -1.5708 0" />
   </joint>
 </robot>

Commit message: updaed launch file, ninjacar urdf, rviz

File: urdf/ninjacar.urdf.xacro (robot description, xacro)
@@ -54,5 +54,6 @@
     <child link="depth_camera_link" />
     <!-- <origin xyz="0.2219971 0 0.130257" rpy="0 0 0" /> -->
-    <origin xyz="0.1143 0 0.13335" rpy="0 0 0" />
+    <!-- <origin xyz="0.1143 0 0.13335" rpy="0 0 0" /> -->
+    <origin xyz="0.1143 0 0." rpy="0 0 0" />
   </joint>
   <link name="royale_camera_link"/>

Commit message: latest experiment setup

File: urdf/ninjacar.urdf.xacro (robot description, xacro)
@@ -55,5 +55,5 @@
     <!-- <origin xyz="0.2219971 0 0.130257" rpy="0 0 0" /> -->
     <!-- <origin xyz="0.1143 0 0.13335" rpy="0 0 0" /> -->
-    <origin xyz="0.1143 0 0." rpy="0 0 0" />
+    <origin xyz="0.1143 0 0.11" rpy="0.01 0 0" />
   </joint>
   <link name="royale_camera_link"/>
@@ -65,5 +65,7 @@
   <xacro:include filename="$(find realsense2_description)/urdf/_d435.urdf.xacro"/>
   <sensor_d435 parent="depth_camera_link" name="d435_camera">
-    <origin xyz="0 0 -0.0127" rpy="0 0 0" />
+    <!-- <origin xyz="0 0 -0.0127" rpy="0 0 0" /> -->
+    <!-- <origin xyz="0 0 0" rpy="0 0 0" /> -->
+    <origin xyz="0 0 0" rpy="$(eval 1*0.0175) $(eval 3.5*0.0175) 0" />
   </sensor_d435>
   <link name="t265_link"/>
